Commit message: Add SAM3D + MANO hand IK (ACADOS MPC), live pipelines, and hand models
- run_ik_acados_mpc_sam3d(_live).py: full-body + MANO finger IK from Goliath-70
- run_ik_live.py / run_ik_live_rerun.py: live retargeting from streamed SAM3D 3D
  (meshcat + optional Rerun mirroring into the extractor's viewer)
- model/: MANO and Sharpa hand URDFs + meshes, human_with_* combined models
- ignore build artifacts (acados/, c_generated_code/, *_ocp.json, output/)

File: model/urdf/1012_scaled.urdf (robot description, URDF)
Before this commit: robot 1012_scaled.urdf, 82 links, 81 joints
Links:
- removed link BHD
- removed link C7
- removed link FHD
- removed link L5MHD
- removed link LANK
- removed link LASI
- removed link LELB
- removed link LHD
- removed link LHEE
- removed link LHM2
- removed link LHM5
- removed link LKNE
- removed link LMANK
- removed link LMELB
- removed link LMKNE
- removed link LMWRI
- removed link LPSI
- removed link LSHO
- removed link LTHI1
- removed link LTIB1
- removed link LTOE
- removed link LWRI
- removed link R5MHD
- removed link RANK
- removed link RASI
- removed link RELB
- removed link RHD
- removed link RHEE
- removed link RHM2
- removed link RHM5
- removed link RKNE
- removed link RMANK
- removed link RMELB
- removed link RMKNE
- removed link RMWRI
- removed link RPSI
- removed link RSHO
- removed link RTHI1
- removed link RTIB1
- removed link RTOE
- removed link RWRI
- removed link SJN
- removed link STRN
- removed link TV12
- removed link TV8
- removed link left_clavicle
- removed link left_foot
- removed link left_foot_virtual
- removed link left_hand
- removed link left_hand_virtual
- removed link left_lowerarm
- removed link left_lowerarm_virtual
- removed link left_lowerleg
- removed link left_upperarm
- removed link left_upperarm_virtual
- removed link left_upperarm_virtual_2
- removed link left_upperleg
- removed link left_upperleg_virtual
- removed link left_upperleg_virtual_2
- removed link middle_abdomen
- removed link middle_abdomen_virtual
- removed link middle_head
- removed link middle_head_virtual
- removed link middle_head_virtual_2
- removed link middle_pelvis
- removed link middle_thorax
- removed link middle_thorax_virtual
- removed link middle_thorax_virtual_2
- removed link right_clavicle
- removed link right_foot
- removed link right_foot_virtual
- removed link right_hand
- removed link right_hand_virtual
- removed link right_lowerarm
- removed link right_lowerarm_virtual
- removed link right_lowerleg
- removed link right_upperarm
- removed link right_upperarm_virtual
- removed link right_upperarm_virtual_2
- removed link right_upperleg
- removed link right_upperleg_virtual
- removed link right_upperleg_virtual_2
- added link right_hand_C_MC, mass 0.6506; collision mesh filename=package://right_sharpa_wave/meshes/right_hand_C_MC.STL; visual mesh filename=package://right_sharpa_wave/meshes/right_hand_C_MC_visual.S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
- added link right_hand_wrist, mass 0.0505; collision mesh filename=package://right_sharpa_wave/meshes/wrist_collision.STL; visual mesh filename=package://right_sharpa_wave/meshes/wrist_B.STL
- added link right_index_DP, mass 0.00455; collision mesh filename=package://right_sharpa_wave/meshes/DP_HB1_4F.STL; visual mesh filename=package://right_sharpa_wave/meshes/DP_visual_HB1_4F.STL
- added link right_index_MCP_VL, mass 2.21E-03; collision mesh filename=package://right_sharpa_wave/meshes/MCP_VL.STL; visual mesh filename=package://right_sharpa_wave/meshes/right_MCP_VL_visual.STL
- added link right_index_MP, mass 0.01824; collision mesh filename=package://right_sharpa_wave/meshes/right_MP.STL; visual mesh filename=package://right_sharpa_wave/meshes/right_MP_visual.STL
- added link right_index_PP, mass 0.04741; collision mesh filename=package://right_sharpa_wave/meshes/right_PP.STL; visual mesh filename=package://right_sharpa_wave/meshes/right_PP_visual.STL
- added link right_index_elastomer, mass 1E-4; collision mesh filename=package://right_sharpa_wave/meshes/elastomer_HB1_4F.STL; visual mesh filename=package://right_sharpa_wave/meshes/elastomer_HB1_4F.STL
- added link right_index_fingertip, mass 1.0E-06
- added link right_middle_DP, mass 0.00455; collision mesh filename=package://right_sharpa_wave/meshes/DP_HB1_4F.STL; visual mesh filename=package://right_sharpa_wave/meshes/DP_visual_HB1_4F.STL
- added link right_middle_MCP_VL, mass 2.21E-03; collision mesh filename=package://right_sharpa_wave/meshes/MCP_VL.STL; visual mesh filename=package://right_sharpa_wave/meshes/right_MCP_VL_visual.STL
- added link right_middle_MP, mass 0.01824; collision mesh filename=package://right_sharpa_wave/meshes/right_MP.STL; visual mesh filename=package://right_sharpa_wave/meshes/right_MP_visual.STL
- added link right_middle_PP, mass 0.04741; collision mesh filename=package://right_sharpa_wave/meshes/right_PP.STL; visual mesh filename=package://right_sharpa_wave/meshes/right_PP_visual.STL
- added link right_middle_elastomer, mass 1E-4; collision mesh filename=package://right_sharpa_wave/meshes/elastomer_HB1_4F.STL; visual mesh filename=package://right_sharpa_wave/meshes/elastomer_HB1_4F.STL
- added link right_middle_fingertip, mass 1.0E-06
- added link right_pinky_DP, mass 0.00455; collision mesh filename=package://right_sharpa_wave/meshes/DP_HB1_4F.STL; visual mesh filename=package://right_sharpa_wave/meshes/DP_visual_HB1_4F.STL
- added link right_pinky_MC, mass 0.12541; collision mesh filename=package://right_sharpa_wave/meshes/right_pinky_MC.STL; visual mesh filename=package://right_sharpa_wave/meshes/right_pinky_MC_visual.STL
- added link right_pinky_MCP_VL, mass 2.21E-03; collision mesh filename=package://right_sharpa_wave/meshes/MCP_VL.STL; visual mesh filename=package://right_sharpa_wave/meshes/right_MCP_VL_visual.STL
- added link right_pinky_MP, mass 0.01824; collision mesh filename=package://right_sharpa_wave/meshes/right_MP.STL; visual mesh filename=package://right_sharpa_wave/meshes/right_MP_visual.STL
- added link right_pinky_PP, mass 0.04741; collision mesh filename=package://right_sharpa_wave/meshes/right_PP.STL; visual mesh filename=package://right_sharpa_wave/meshes/right_PP_visual.STL
- added link right_pinky_elastomer, mass 1E-4; collision mesh filename=package://right_sharpa_wave/meshes/elastomer_HB1_4F.STL; visual mesh filename=package://right_sharpa_wave/meshes/elastomer_HB1_4F.STL
- added link right_pinky_fingertip, mass 1.0E-06
- added link right_ring_DP, mass 0.00455; collision mesh filename=package://right_sharpa_wave/meshes/DP_HB1_4F.STL; visual mesh filename=package://right_sharpa_wave/meshes/DP_visual_HB1_4F.STL
- added link right_ring_MCP_VL, mass 2.21E-03; collision mesh filename=package://right_sharpa_wave/meshes/MCP_VL.STL; visual mesh filename=package://right_sharpa_wave/meshes/right_MCP_VL_visual.STL
- added link right_ring_MP, mass 0.01824; collision mesh filename=package://right_sharpa_wave/meshes/right_MP.STL; visual mesh filename=package://right_sharpa_wave/meshes/right_MP_visual.STL
- added link right_ring_PP, mass 0.04741; collision mesh filename=package://right_sharpa_wave/meshes/right_PP.STL; visual mesh filename=package://right_sharpa_wave/meshes/right_PP_visual.STL
- added link right_ring_elastomer, mass 1E-4; collision mesh filename=package://right_sharpa_wave/meshes/elastomer_HB1_4F.STL; visual mesh filename=package://right_sharpa_wave/meshes/elastomer_HB1_4F.STL
- added link right_ring_fingertip, mass 1.0E-06
- added link right_thumb_CMC_VL, mass 2.5E-03; visual mesh filename=package://right_sharpa_wave/meshes/right_thumb_CMC_VL_visua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
- added link right_thumb_DP, mass 0.00788; collision mesh filename=package://right_sharpa_wave/meshes/DP_HB1_TH.STL; visual mesh filename=package://right_sharpa_wave/meshes/DP_Visual_HB1_TH.STL
- added link right_thumb_MC, mass 0.13587; collision mesh filename=package://right_sharpa_wave/meshes/right_thumb_MC.STL; visual mesh filename=package://right_sharpa_wave/meshes/right_thumb_MC_visual.STL
- added link right_thumb_MCP_VL, mass 8E-5; visual mesh filename=package://right_sharpa_wave/meshes/right_thumb_MCP_VL_visua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
- added link right_thumb_PP, mass 0.03078; collision mesh filename=package://right_sharpa_wave/meshes/right_thumb_PP.STL; visual mesh filename=package://right_sharpa_wave/meshes/right_thumb_PP_visual.STL
- added link right_thumb_elastomer, mass 1E-4; collision mesh filename=package://right_sharpa_wave/meshes/elastomer_HB1_TH.STL; visual mesh filename=package://right_sharpa_wave/meshes/elastomer_HB1_TH.STL
- added link right_thumb_fingertip, mass 1.0E-06
Joints:
- removed joint joint_BHD
- removed joint joint_C7
- removed joint joint_FHD
- removed joint joint_L5MHD
- removed joint joint_LANK
- removed joint joint_LASI
- removed joint joint_LELB
- removed joint joint_LHD
- removed joint joint_LHEE
- removed joint joint_LHM2
- removed joint joint_LHM5
- removed joint joint_LKNE
- removed joint joint_LMANK
- removed joint joint_LMELB
- removed joint joint_LMKNE
- removed joint joint_LMWRI
- removed joint joint_LPSI
- removed joint joint_LSHO
- removed joint joint_LTHI1
- removed joint joint_LTIB1
- removed joint joint_LTOE
- removed joint joint_LWRI
- removed joint joint_R5MHD
- removed joint joint_RANK
- removed joint joint_RASI
- removed joint joint_RELB
- removed joint joint_RHD
- removed joint joint_RHEE
- removed joint joint_RHM2
- removed joint joint_RHM5
- removed joint joint_RKNE
- removed joint joint_RMANK
- removed joint joint_RMELB
- removed joint joint_RMKNE
- removed joint joint_RMWRI
- removed joint joint_RPSI
- removed joint joint_RSHO
- removed joint joint_RTHI1
- removed joint joint_RTIB1
- removed joint joint_RTOE
- removed joint joint_RWRI
- removed joint joint_SJN
- removed joint joint_STRN
- removed joint joint_TV12
- removed joint joint_TV8
- removed joint left_ankle_X
- removed joint left_ankle_Z
- removed joint left_clavicle_joint_X
- removed joint left_elbow_Y
- removed joint left_elbow_Z
- removed joint left_hip_X
- removed joint left_hip_Y
- removed joint left_hip_Z
- removed joint left_knee_Z
- removed joint left_shoulder_X
- removed joint left_shoulder_Y
- removed joint left_shoulder_Z
- removed joint left_wrist_X
- removed joint left_wrist_Z
- removed joint middle_cervical_X
- removed joint middle_cervical_Y
- removed joint middle_cervical_Z
- removed joint middle_lumbar_X
- removed joint middle_lumbar_Z
- removed joint middle_thoracic_X
- removed joint middle_thoracic_Y
- removed joint middle_thoracic_Z
- removed joint right_ankle_X
- removed joint right_ankle_Z
- removed joint right_clavicle_joint_X
- removed joint right_elbow_Y
- removed joint right_elbow_Z
- removed joint right_hip_X
- removed joint right_hip_Y
- removed joint right_hip_Z
- removed joint right_knee_Z
- removed joint right_shoulder_X
- removed joint right_shoulder_Y
- removed joint right_shoulder_Z
- removed joint right_wrist_X
- removed joint right_wrist_Z
- added joint right_hand_wrist_fix_joint: type fixed, parent right_hand_wrist, child right_hand_C_MC, origin xyz=0 0 0.029 rpy=0 0 0, axis 0 0 0
- added joint right_index_DIP: type revolute, parent right_index_MP, child right_index_DP, origin xyz=0.0262736 0 0 rpy=0 0 0, axis 0 0 1, limit lower=0 upper=1.3963 effort=0.189369 velocity=14.66594768
- added joint right_index_MCP_AA: type revolute, parent right_index_MCP_VL, child right_index_PP, origin xyz=0 0 0 rpy=-1.5708 0 0, axis 0 0 1, limit lower=-0.3491 upper=0.3491 effort=1.864 velocity=16.07692878
- added joint right_index_MCP_FE: type revolute, parent right_hand_C_MC, child right_index_MCP_VL, origin xyz=0.001 0.0303 0.0903549 rpy=0 -1.5708 -1.5708, axis 0 0 1, limit lower=-0.17453293 upper=1.5708 effort=1.864 velocity=16.07692878
- added joint right_index_PIP: type revolute, parent right_index_PP, child right_index_MP, origin xyz=0.0405349 0 0 rpy=1.5708 0 0, axis 0 0 1, limit lower=0 upper=1.7453 effort=0.638 velocity=11.61831603
- added joint right_index_elastomer_fix_joint: type fixed, parent right_index_DP, child right_index_elastomer, origin xyz=0 0 0 rpy=1.5708 -1.5708 0, axis 0 0 0
- added joint right_index_fingertip_fix_joint: type fixed, parent right_index_elastomer, child right_index_fingertip, origin xyz=0 -0.0228821 0 rpy=1.5708 1.5708 0, axis 0 0 0
- added joint right_middle_DIP: type revolute, parent right_middle_MP, child right_middle_DP, origin xyz=0.0282131 0 0 rpy=0 0 0, axis 0 0 1, limit lower=0 upper=1.3963 effort=0.189369 velocity=14.66594768
- added joint right_middle_MCP_AA: type revolute, parent right_middle_MCP_VL, child right_middle_PP, origin xyz=0 0 0 rpy=-1.5708 0 0, axis 0 0 1, limit lower=-0.3491 upper=0.3491 effort=1.864 velocity=16.07692878
- added joint right_middle_MCP_FE: type revolute, parent right_hand_C_MC, child right_middle_MCP_VL, origin xyz=0 0.01 0.0881804 rpy=0 -1.5708 -1.5708, axis 0 0 1, limit lower=-0.17453293 upper=1.5708 effort=1.864 velocity=16.07692878
- added joint right_middle_PIP: type revolute, parent right_middle_PP, child right_middle_MP, origin xyz=0.0450564 0 0 rpy=1.5708 0 0, axis 0 0 1, limit lower=0 upper=1.7453 effort=0.638 velocity=11.61831603
- added joint right_middle_elastomer_fix_joint: type fixed, parent right_middle_DP, child right_middle_elastomer, origin xyz=0 0 0 rpy=1.5707963267949 -1.5707963267949 0, axis 0 0 0
- added joint right_middle_fingertip_fix_joint: type fixed, parent right_middle_elastomer, child right_middle_fingertip, origin xyz=0 -0.0235861 0 rpy=1.5707963267949 1.5707963267949 0, axis 0 0 0
- added joint right_pinky_CMC: type revolute, parent right_hand_C_MC, child right_pinky_MC, origin xyz=0.01136 -0.0263 0.0796983 rpy=0 0 3.1416, axis 0 0 1, limit lower=0 upper=0.2618 effort=0.5285 velocity=35.07416159
- added joint right_pinky_DIP: type revolute, parent right_pinky_MP, child right_pinky_DP, origin xyz=0.0215545 0 0 rpy=0 0 0, axis 0 0 1, limit lower=0 upper=1.3963 effort=0.189369 velocity=14.66594768
- added joint right_pinky_MCP_AA: type revolute, parent right_pinky_MCP_VL, child right_pinky_PP, origin xyz=0 0 0 rpy=-1.5708 0 0, axis 0 0 1, limit lower=-0.3491 upper=0.3491 effort=1.864 velocity=16.07692878
- added joint right_pinky_MCP_FE: type revolute, parent right_pinky_MC, child right_pinky_MCP_VL, origin xyz=0.00836 0.0048 0 rpy=1.5708 -1.5708 0, axis 0 0 1, limit lower=-0.17453293 upper=1.5708 effort=1.864 velocity=16.07692878
- added joint right_pinky_PIP: type revolute, parent right_pinky_PP, child right_pinky_MP, origin xyz=0.032025 0 0 rpy=1.5708 0 0, axis 0 0 1, limit lower=0 upper=1.7453 effort=0.638 velocity=11.61831603
- added joint right_pinky_elastomer_fix_joint: type fixed, parent right_pinky_DP, child right_pinky_elastomer, origin xyz=0 0 0 rpy=1.5708 -1.5708 0, axis 0 0 0
- added joint right_pinky_fingertip_fix_joint: type fixed, parent right_pinky_elastomer, child right_pinky_fingertip, origin xyz=0 -0.0208725 0 rpy=1.5708 1.5708 0, axis 0 0 0
- added joint right_ring_DIP: type revolute, parent right_ring_MP, child right_ring_DP, origin xyz=0.0280232 0 0 rpy=0 0 0, axis 0 0 1, limit lower=0 upper=1.3963 effort=0.189369 velocity=14.66594768
- added joint right_ring_MCP_AA: type revolute, parent right_ring_MCP_VL, child right_ring_PP, origin xyz=0 0 0 rpy=-1.5708 0 0, axis 0 0 1, limit lower=-0.3491 upper=0.3491 effort=1.864 velocity=16.07692878
- added joint right_ring_MCP_FE: type revolute, parent right_hand_C_MC, child right_ring_MCP_VL, origin xyz=0.0015 -0.0103 0.0826864 rpy=0 -1.5708 -1.5708, axis 0 0 1, limit lower=-0.17453293 upper=1.5708 effort=1.864 velocity=16.07692878
- added joint right_ring_PIP: type revolute, parent right_ring_PP, child right_ring_MP, origin xyz=0.0413558 0 0 rpy=1.5708 0 0, axis 0 0 1, limit lower=0 upper=1.7453 effort=0.638 velocity=11.61831603
- added joint right_ring_elastomer_fix_joint: type fixed, parent right_ring_DP, child right_ring_elastomer, origin xyz=0 0 0 rpy=1.5708 -1.5708 0, axis 0 0 0
- added joint right_ring_fingertip_fix_joint: type fixed, parent right_ring_elastomer, child right_ring_fingertip, origin xyz=0 -0.0235312 0 rpy=1.5707963267949 1.5707963267949 0, axis 0 0 0
- added joint right_thumb_CMC_AA: type revolute, parent right_thumb_CMC_VL, child right_thumb_MC, origin xyz=0 -0.005 0 rpy=-1.5708 0.7854 0, axis 0 0 1, limit lower=-0.3491 upper=0.3491 effort=3.3 velocity=11.84076833
- added joint right_thumb_CMC_FE: type revolute, parent right_hand_C_MC, child right_thumb_CMC_VL, origin xyz=0.0121295 0.0315367 0.0259571 rpy=3.1416 0 1.5708, axis 0 0 1, limit lower=-0.1745 upper=1.9199 effort=3.3 velocity=11.84076833
- added joint right_thumb_IP: type revolute, parent right_thumb_PP, child right_thumb_DP, origin xyz=0.0363373 0 0 rpy=1.5708 0 0, axis 0 0 1, limit lower=0 upper=1.7453 effort=0.638 velocity=11.61831603
- added joint right_thumb_MCP_AA: type revolute, parent right_thumb_MCP_VL, child right_thumb_PP, origin xyz=0 0 0 rpy=-1.5708 0 0, axis 0 0 1, limit lower=-0.3491 upper=0.3491 effort=1.864 velocity=16.07692878
- added joint right_thumb_MCP_FE: type revolute, parent right_thumb_MC, child right_thumb_MCP_VL, origin xyz=0.0345606 -0.006 0.010392 rpy=0.5236 0 0, axis 0 0 1, limit lower=-0.5236 upper=1.3963 effort=1.864 velocity=16.07692878
- added joint right_thumb_elastomer_fix_joint: type fixed, parent right_thumb_DP, child right_thumb_elastomer, origin xyz=0 0 0 rpy=1.5708 -1.5708 0, axis 0 0 0
- added joint right_thumb_fingertip_fix_joint: type fixed, parent right_thumb_elastomer, child right_thumb_fingertip, origin xyz=0 -0.0278606 0 rpy=1.5708 1.5708 0, axis 0 0 0
